Commit message: fixed propeller lift params

File: urdf/drone.urdf (robot description, URDF)
Before this commit: robot drone_description, 7 links, 6 joints
Joints:
- joint back_left_prop_joint: axis 0 0 1 -> 0 0 -1
- joint front_right_prop_joint: axis 0 0 1 -> 0 0 -1

File: urdf/drone_base.xacro (robot description, xacro)
@@ -5,6 +5,5 @@
   <xacro:include filename="$(find drone_description)/urdf/drone_macros.xacro" />
   <xacro:include filename="$(find drone_description)/urdf/drone_gazebo.xacro" />
-  <xacro:include filename="$(find drone_description)/urdf/sensors/camera.xacro" />
-  <!-- <xacro:include filename="$(find drone_description)/urdf/sensors/force.xacro" /> -->
+  <xacro:include filename="$(find drone_description)/urdf/sensors.xacro" />
   <!-- DUMMY lINK -->
   <link name="dummy_link" />
@@ -64,7 +63,17 @@
     <parent link="base_link" />
     <child link="camera" />
-    <axis xyz="0 0 -1" />
-    <limit lower="-${PI/3}" upper="0" effort="0" velocity="0" />
+    <axis xyz="0 0 1" />
+    <limit lower="0" upper="${PI/3}" effort="100" velocity="1" />
   </joint>
+  <transmission name="camera_trans">
+    <type>transmission_interface/SimpleTransmission</type>
+    <joint name="camera_joint">
+      <hardwareInterface>hardware_interface/PositionJointInterface</hardwareInterface>
+    </joint>
+    <actuator name="camera_motor">
+      <mechanicalReduction>1</mechanicalReduction>
+      <hardwareInterface>hardware_interface/PositionJointInterface</hardwareInterface>
+    </actuator>
+  </transmission>
   <xacro:prop_link name="front_left_prop" />
   <xacro:prop_link name="front_right_prop" />
@@ -79,7 +88,7 @@
   <xacro:prop_transmission name="back_left_prop" />
   <xacro:prop_transmission name="back_right_prop" />
-  <!-- <xacro:propeller_plugin name="front_left_prop" dir="1" />
-  <xacro:propeller_plugin name="front_right_prop" dir="-1" />
-  <xacro:propeller_plugin name="back_left_prop" dir="-1" />
-  <xacro:propeller_plugin name="back_right_prop" dir="1" /> -->
+  <xacro:propeller_plugin name="front_left_prop" dir="-1" />
+  <xacro:propeller_plugin name="front_right_prop" dir="1" />
+  <xacro:propeller_plugin name="back_left_prop" dir="1" />
+  <xacro:propeller_plugin name="back_right_prop" dir="-1" />
 </robot>

File: urdf/drone_gazebo.xacro (robot description, xacro)
@@ -7,20 +7,21 @@
     </plugin>
   </gazebo>
-  <!-- lIFT DRAG -->
+  <!-- LIFT DRAG -->
   <xacro:macro name="propeller_plugin" params="name dir">
     <gazebo>
-      <plugin name="${name}_lift" filename="libliftDragPlugin.so">
+      <!-- Provide a Positive Velocity -->
+      <plugin name="${name}_lift" filename="libLiftDragPlugin.so">
         <a0>0.1</a0>
         <cla>0.1</cla>
         <cda>0.01</cda>
         <cma>0.0</cma>
-        <alpha_stall>0.3368</alpha_stall>
-        <cla_stall>-2.1419</cla_stall>
-        <cda_stall>0.0</cda_stall>
+        <alpha_stall>1.0472</alpha_stall>
+        <cla_stall>-0.2</cla_stall>
+        <cda_stall>1.0</cda_stall>
         <cma_stall>0.0</cma_stall>
         <cp>0 0.5 0</cp>
-        <area>0.01</area>
+        <area>0.70</area>
         <air_density>1.2041</air_density>
-        <forward>-1 0 0</forward>
+        <forward>1 0 0</forward>
         <upward>0 0 ${dir}</upward>
         <link_name>${name}</link_name>

File: urdf/drone_macros.xacro (robot description, xacro)
@@ -45,13 +45,3 @@
     </transmission>
   </xacro:macro>
-  <!-- <transmission name="camera">
-    <type>transmission_interface/SimpleTransmission</type>
-    <joint name="camera_joint">
-      <hardwareInterface>hardware_interface/PositionJointInterface</hardwareInterface>
-    </joint>
-    <actuator name="camera_motor">
-      <mechanicalReduction>1</mechanicalReduction>
-      <hardwareInterface>hardware_interface/PositionJointInterface</hardwareInterface>
-    </actuator>
-  </transmission> -->
 </robot>

File: urdf/sensors.xacro (robot description, xacro)
@@ -1,4 +1,25 @@
 <?xml version="1.0" encoding="UTF-8"?>
-<robot xmlns:xacro="http://www.ros.org/wiki/xacro">
+<robot xmlns:xacro="www.ros.org/wiki/xacro">
+  <!-- IMU -->
+  <gazebo reference="base_link">
+    <gravity>true</gravity>
+    <sensor name="imu_sensor" type="imu">
+      <always_on>true</always_on>
+      <update_rate>100</update_rate>
+      <visualize>true</visualize>
+      <topic>__default_topic__</topic>
+      <plugin filename="libgazebo_ros_imu_sensor.so" name="imu_plugin">
+        <topicName>imu</topicName>
+        <bodyName>base_link</bodyName>
+        <updateRateHZ>10.0</updateRateHZ>
+        <gaussianNoise>0.0</gaussianNoise>
+        <xyzOffset>0 0 0</xyzOffset>
+        <rpyOffset>0 0 0</rpyOffset>
+        <frameName>base_link</frameName>
+        <initialOrientationAsReference>false</initialOrientationAsReference>
+      </plugin>
+      <pose>0 0 0 0 0 0</pose>
+    </sensor>
+  </gazebo>
   <!-- CAMERA -->
   <gazebo reference="camera">
